File: BE_elec.kicad_pcb (KiCad board)
At the start: 2 copper layers, 110 x 100 mm, 54 parts, among them J2 Conn_01x02, J3 Conn_01x03, Q1 2N2907, Q10 TIP32, Q11 BD138, Q12 TIP31, Q13 2N222, Q2 2N2907, Q3 2N2907, Q4 2N222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

Commit message: -all
Parts:
- moved C6 196.9 mm to (38.1, 39.4)
- moved C5 194.7 mm to (22.9, 48.3)
- moved C4 188.2 mm to (22.9, 39.4)
- moved Q1 171.2 mm to (68.6, 43.2)
- moved C7 170.7 mm to (38.1, 48.3)
- moved D4 162.0 mm to (36.8, 30.5)
- moved C1 155.2 mm to (67.3, 33.0)
- moved D3 146.4 mm to (20.3, 30.5)
- moved Q2 142.6 mm to (78.7, 43.2)
- moved R1 106.5 mm to (78.7, 35.6)
- moved R2 99.5 mm to (92.7, 35.6)
- moved R3 81.5 mm to (108.0, 35.6)
- moved U1 25.3 mm to (160.0, 33.0)
- moved J2 14.8 mm to (94.0, 20.9), turned to 180 degrees
- moved J3 7.54 mm to (53.3, 21.6), turned to 180 degrees
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
Commit message: --all
Parts:
- moved HS1 222.7 mm to (50.8, 34.3)
- moved Q4 213.4 mm to (24.1, 69.8)
- moved C2 204.0 mm to (24.1, 55.9), turned to 270 degrees
- moved RV1 201.4 mm to (24.1, 38.1), turned to 180 degrees
- moved Q3 191.0 mm to (38.1, 82.5), turned to 180 degrees
- moved Q6 187.1 mm to (40.6, 48.3)
- moved Q5 178.9 mm to (33.0, 62.1), turned to 270 degrees
- moved Q7 176.5 mm to (47.0, 63.5), turned to 270 degrees
- moved Q8 174.3 mm to (22.9, 48.3)
- moved Q9 174.3 mm to (21.6, 25.4), turned to 270 degrees
- moved R10 172.2 mm to (48.3, 50.8)
- moved Dz1 168.7 mm to (59.7, 94.0), turned to 180 degrees
- moved C9 168.3 mm to (61.0, 61.0), turned to 180 degrees
- moved HS2 164.4 mm to (106.7, 64.8)
- moved R7 159.2 mm to (45.7, 73.7), turned to 180 degrees
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