File: BE_elec.kicad_pcb (KiCad board)
At the start: 2 copper layers, 110 x 100 mm, 54 parts, among them J2 Conn_01x02, J3 Conn_01x03, Q1 2N2907, Q10 TIP32, Q11 BD138, Q12 TIP31, Q13 2N222, Q2 2N2907, Q3 2N2907, Q4 2N222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

Commit message: Mise à jour netlist et dernières modifications de placement.
Parts:
- Q13: footprint CmpAmpliAudio:TO-92_Inline_Wide -> CmpAmpliAudio:TO-18-3
- moved HS1 215.2 mm to (54.6, 47.0), turned to 90 degrees
- moved Q6 205.1 mm to (20.3, 88.9)
- moved C9 204.4 mm to (25.4, 44.5), turned to 180 degrees
- moved Q7 203.3 mm to (19.1, 100.3)
- moved R10 194.9 mm to (36.8, 111.8)
- moved C2 189.9 mm to (39.4, 87.6)
- moved Q4 184.4 mm to (54.6, 91.4), turned to 270 degrees
- moved R7 177.4 mm to (29.2, 88.9), turned to 270 degrees
- moved RV1 176.0 mm to (49.5, 78.7)
- moved HS2 164.9 mm to (116.8, 41.9), turned to 90 degrees
- moved C8 163.0 mm to (20.3, 31.8)
- moved Q8 162.0 mm to (29.2, 81.3)
- moved R9 159.3 mm to (34.3, 94.0), turned to 270 degrees
- moved RV2 156.7 mm to (47.0, 104.1)
- moved Dz1 155.4 mm to (76.2, 100.3)
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
Commit message: Inversion pistes relai
Parts:
- moved R12 17.8 mm to (102.9, 34.3), turned to 270 degrees
- moved Q6 10.9 mm to (26.7, 97.8), turned to 90 degrees
- moved R7 10.2 mm to (19.1, 87.6)
- moved C3 6.48 mm to (91.4, 69.8), turned to 180 degrees
- moved Q8 5.68 mm to (34.3, 83.8), turned to 90 degrees
- moved Q2 5.39 mm to (114.3, 104.1)
- moved Q7 5.39 mm to (22.9, 104.1), turned to 270 degrees
- moved R8 5.24 mm to (49.5, 73.7)
- moved Q9 4.02 mm to (44.5, 66.0), turned to 270 degrees
- moved Q13 3.59 mm to (74.9, 63.5), turned to 270 degrees
Routing:
- net GND: track 0.00 -> 316.5 mm
- net -12V: track 0.00 -> 271.9 mm
- net +12V: track 0.00 -> 250.2 mm
- net Net-(C2-Pad1): track 0.00 -> 127.1 mm
- net Net-(R11-Pad2): track 0.00 -> 126.6 mm
- net Net-(Q5-Pad1): track 0.00 -> 79.2 mm
- net Net-(C2-Pad2): track 0.00 -> 78.8 mm
- net Net-(Q2-Pad2): track 0.00 -> 65.6 mm
- net Net-(Q6-Pad3): track 0.00 -> 56.5 mm
- net Net-(Q10-Pad2): track 0.00 -> 43.4 mm
- net Net-(C1-Pad2): track 0.00 -> 33.4 mm
- net Net-(Q1-Pad1): track 0.00 -> 33.0 mm
- net Net-(Q11-Pad2): track 0.00 -> 32.7 mm
- net Net-(D2-Pad1): track 0.00 -> 31.7 mm
- net Net-(C1-Pad1): track 0.00 -> 30.9 mm
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Other:
- board text added: "Bottom Jullien Galloo"
- board text added: "Face Jullien Galloo"
