File: BE_Elec_Final.kicad_pcb (KiCad board)
At the start: 2 copper layers, 110 x 100 mm, 54 parts, among them J2 Conn_01x02, J3 Conn_01x03, Q1 2N2907, Q10 TIP32, Q11 BD138, Q12 TIP31, Q13 2N222, Q2 2N2907, Q3 2N2907, Q4 2N222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

Commit message: bug
Parts:
- Q13: footprint CmpAmpliAudio:TO-18-3 -> CmpAmpliAudio:TO-92_Inline_Wide
- moved R11 33.0 mm to (35.6, 27.9)
- moved R12 17.8 mm to (102.9, 52.1), turned to 90 degrees
- moved Q6 10.9 mm to (20.3, 88.9), turned to 0 degrees
- moved R7 10.2 mm to (29.2, 88.9)
- moved C3 6.48 mm to (85.1, 68.6), turned to 0 degrees
- moved Q8 5.68 mm to (29.2, 81.3), turned to 0 degrees
- moved Q2 5.39 mm to (110.5, 108.0)
- moved Q7 5.39 mm to (19.1, 100.3), turned to 0 degrees
- moved R8 5.24 mm to (54.6, 74.9)
- moved J2 5.13 mm to (94.0, 20.9), turned to 180 degrees
- moved Q9 4.02 mm to (45.7, 69.8), turned to 0 degrees
- moved Q13 3.59 mm to (77.5, 66.0), turned to 180 degrees
- moved U1 2.54 mm to (69.8, 55.9)
- moved HS1 2.54 mm to (57.1, 47.0)
- moved Q12 1.27 mm to (110.5, 39.4)
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Routing:
- net Net-(C2-Pad1): track 339.1 -> 0.00 mm
- net GND: track 311.6 -> 0.00 mm
- net -12V: track 270.3 -> 0.00 mm
- net +12V: track 245.4 -> 0.00 mm
- net Net-(R11-Pad2): track 126.6 -> 0.00 mm
- net Net-(Q5-Pad1): track 79.2 -> 0.00 mm
- net Net-(C2-Pad2): track 78.8 -> 0.00 mm
- net Net-(Q2-Pad2): track 61.6 -> 0.00 mm
- net Net-(Q6-Pad3): track 56.5 -> 0.00 mm
- net Net-(Q10-Pad2): track 43.4 -> 0.00 mm
- net Net-(C1-Pad2): track 33.4 -> 0.00 mm
- net Net-(D2-Pad1): track 31.7 -> 0.00 mm
- net Net-(C1-Pad1): track 30.9 -> 0.00 mm
- net Net-(Q6-Pad2): track 30.6 -> 0.00 mm
- net Net-(Q1-Pad1): track 30.2 -> 0.00 mm
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Other:
- board text removed: "Bottom Jullien Galloo"
- board text removed: "Face Jullien Galloo"
