File: BE_Elec.sch (KiCad schematic (older format))
At the start: 51 parts, among them J2 Conn_01x02, J3 Conn_01x03, Q1 2N2907, Q10 TIP32, Q11 BD138, Q12 TIP31, Q13 2N222, Q2 2N2907, Q3 2N2907, Q4 2N222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

Commit message: --all
Parts:
- added U1: Relay_1CT, BE_Elec:Relay_1CT, symbol be-elec:Relay_1CT
- R1, R10, R11, R12, R13, R14, R15, R16, R17, R2, R3, R4, R5, R6, R7, R8, R9: footprint (none) -> CmpAmpliAudio:R_Axial_DIN0207_L6.3mm_D2.5mm_P10.16mm_Horizontal
- RV1, RV2: footprint (none) -> CmpAmpliAudio:R_Axial_DIN0516_L15.5mm_D5.0mm_P20.32mm_Horizontal
- U2: footprint (none) -> CmpAmpliAudio:Jack_35RAPC2AV; symbol CmpAmpliAudio:Jack_Mono -> BE_Elec-rescue:Jack_Mono-CmpAmpliAudio
Connections:
- wire segments 169 -> 168
Changed lines of the file:
@@
 $EndDescr
 $Comp
-L CmpAmpliAudio:Jack_Mono U2
+L BE_Elec-rescue:Jack_Mono-CmpAmpliAudio U2
 U 1 1 60591E24
 P 950 3350
 F 0 "U2" H 978 3617 50  0000 C CNN
 F 1 "Jack_Mono" H 978 3526 50  0000 C CNN
-F 2 "" H 1000 3550 50  0001 C CNN
+F 2 "CmpAmpliAudio:Jack_35RAPC2AV" H 1000 3550 50  0001 C CNN
 F 3 "" H 1000 3550 50  0001 C CNN
 	1    950  3350
@@
 F 0 "R1" H 2070 3846 50  0000 L CNN
 F 1 "R" H 2070 3755 50  0000 L CNN
-F 2 "" V 1930 3800 50  0001 C CNN
+F 2 "CmpAmpliAudio:R_Axial_DIN0207_L6.3mm_D2.5mm_P10.16mm_Horizontal" V 1930 3800 50  0001 C CNN
 F 3 "~" H 2000 3800 50  0001 C CNN
 	1    2000 3800
@@
 F 0 "R5" H 2320 2496 50  0000 L CNN
 F 1 "R" H 2320 2405 50  0000 L CNN
-F 2 "" V 2180 2450 50  0001 C CNN
+F 2 "CmpAmpliAudio:R_Axial_DIN0207_L6.3mm_D2.5mm_P10.16mm_Horizontal" V 2180 2450 50  0001 C CNN
 F 3 "~" H 2250 2450 50  0001 C CNN
 	1    2250 2450
@@
 F 0 "R4" H 2970 1646 50  0000 L CNN
 F 1 "R" H 2970 1555 50  0000 L CNN
-F 2 "" V 2830 1600 50  0001 C CNN
+F 2 "CmpAmpliAudio:R_Axial_DIN0207_L6.3mm_D2.5mm_P10.16mm_Horizontal" V 2830 1600 50  0001 C CNN
 F 3 "~" H 2900 1600 50  0001 C CNN
 	1    2900 1600
@@
 F 0 "R2" H 2620 4096 50  0000 L CNN
 F 1 "R" H 2620 4005 50  0000 L CNN
-F 2 "" V 2480 4050 50  0001 C CNN
+F 2 "CmpAmpliAudio:R_Axial_DIN0207_L6.3mm_D2.5mm_P10.16mm_Horizontal" V 2480 4050 50  0001 C CNN
 F 3 "~" H 2550 4050 50  0001 C CNN
 	1    2550 4050
@@
 F 0 "R3" H 3420 4096 50  0000 L CNN
 F 1 "R" H 3420 4005 50  0000 L CNN
-F 2 "" V 3280 4050 50  0001 C CNN
+F 2 "CmpAmpliAudio:R_Axial_DIN0207_L6.3mm_D2.5mm_P10.16mm_Horizontal" V 3280 4050 50  0001 C CNN
 F 3 "~" H 3350 4050 50  0001 C CNN
 	1    3350 4050
@@
 F 0 "R15" H 4020 5296 50  0000 L CNN
 F 1 "R" H 4020 5205 50  0000 L CNN
-F 2 "" V 3880 5250 50  0001 C CNN
+F 2 "CmpAmpliAudio:R_Axial_DIN0207_L6.3mm_D2.5mm_P10.16mm_Horizontal" V 3880 5250 50  0001 C CNN
 F 3 "~" H 3950 5250 50  0001 C CNN
 	1    3950 5250
@@
 F 0 "R6" H 5170 4546 50  0000 L CNN
 F 1 "R" H 5170 4455 50  0000 L CNN
-F 2 "" V 5030 4500 50  0001 C CNN
+F 2 "CmpAmpliAudio:R_Axial_DIN0207_L6.3mm_D2.5mm_P10.16mm_Horizontal" V 5030 4500 50  0001 C CNN
 F 3 "~" H 5100 4500 50  0001 C CNN
 	1    5100 4500
@@
 F 0 "R8" H 4820 2996 50  0000 L CNN
 F 1 "R" H 4820 2905 50  0000 L CNN
-F 2 "" V 4680 2950 50  0001 C CNN
+F 2 "CmpAmpliAudio:R_Axial_DIN0207_L6.3mm_D2.5mm_P10.16mm_Horizontal" V 4680 2950 50  0001 C CNN
 F 3 "~" H 4750 2950 50  0001 C CNN
 	1    4750 2950
@@
 F 0 "RV1" H 4431 2646 50  0000 R CNN
 F 1 "R_POT" H 4431 2555 50  0000 R CNN
-F 2 "" H 4500 2600 50  0001 C CNN
+F 2 "CmpAmpliAudio:R_Axial_DIN0516_L15.5mm_D5.0mm_P20.32mm_Horizontal" H 4500 2600 50  0001 C CNN
 F 3 "~" H 4500 2600 50  0001 C CNN
 	1    4500 2600
@@
 F 0 "R7" H 5170 1546 50  0000 L CNN
 F 1 "R" H 5170 1455 50  0000 L CNN
-F 2 "" V 5030 1500 50  0001 C CNN
+F 2 "CmpAmpliAudio:R_Axial_DIN0207_L6.3mm_D2.5mm_P10.16mm_Horizontal" V 5030 1500 50  0001 C CNN
 F 3 "~" H 5100 1500 50  0001 C CNN
 	1    5100 1500
@@
 F 0 "R9" H 4020 1546 50  0000 L CNN
 F 1 "R" H 4020 1455 50  0000 L CNN
-F 2 "" V 3880 1500 50  0001 C CNN
+F 2 "CmpAmpliAudio:R_Axial_DIN0207_L6.3mm_D2.5mm_P10.16mm_Horizontal" V 3880 1500 50  0001 C CNN
 F 3 "~" H 3950 1500 50  0001 C CNN
 	1    3950 1500
@@
 F 0 "R10" H 4020 2546 50  0000 L CNN
 F 1 "R" H 4020 2455 50  0000 L CNN
-F 2 "" V 3880 2500 50  0001 C CNN
+F 2 "CmpAmpliAudio:R_Axial_DIN0207_L6.3mm_D2.5mm_P10.16mm_Horizontal" V 3880 2500 50  0001 C CNN
 F 3 "~" H 3950 2500 50  0001 C CNN
 	1    3950 2500
@@
 F 0 "RV2" H 3880 2904 50  0000 R CNN
 F 1 "R_POT" H 3880 2995 50  0000 R CNN
-F 2 "" H 3950 2950 50  0001 C CNN
+F 2 "CmpAmpliAudio:R_Axial_DIN0516_L15.5mm_D5.0mm_P20.32mm_Horizontal" H 3950 2950 50  0001 C CNN
 F 3 "~" H 3950 2950 50  0001 C CNN
 	1    3950 2950
@@
 F 0 "R11" H 6470 2846 50  0000 L CNN
 F 1 "R" H 6470 2755 50  0000 L CNN
-F 2 "" V 6330 2800 50  0001 C CNN
+F 2 "CmpAmpliAudio:R_Axial_DIN0207_L6.3mm_D2.5mm_P10.16mm_Horizontal" V 6330 2800 50  0001 C CNN
 F 3 "~" H 6400 2800 50  0001 C CNN
 	1    6400 2800
@@
 F 0 "R12" H 6470 3346 50  0000 L CNN
 F 1 "R" H 6470 3255 50  0000 L CNN
-F 2 "" V 6330 3300 50  0001 C CNN
+F 2 "CmpAmpliAudio:R_Axial_DIN0207_L6.3mm_D2.5mm_P10.16mm_Horizontal" V 6330 3300 50  0001 C CNN
 F 3 "~" H 6400 3300 50  0001 C CNN
 	1    6400 3300
@@
 F 0 "R14" V 4700 5000 50  0000 L CNN
 F 1 "R" V 4620 5005 50  0000 L CNN
-F 2 "" V 4480 5050 50  0001 C CNN
+F 2 "CmpAmpliAudio:R_Axial_DIN0207_L6.3mm_D2.5mm_P10.16mm_Horizontal" V 4480 5050 50  0001 C CNN
 F 3 "~" H 4550 5050 50  0001 C CNN
 	1    4550 5050
@@
 Wire Wire Line
 	5100 4850 6400 4850
-Wire Wire Line
-	6400 4850 6400 4800
 Connection ~ 5100 4850
 Wire Wire Line
@@
 F 0 "R13" H 7420 3396 50  0000 L CNN
 F 1 "R" H 7420 3305 50  0000 L CNN
-F 2 "" V 7280 3350 50  0001 C CNN
+F 2 "CmpAmpliAudio:R_Axial_DIN0207_L6.3mm_D2.5mm_P10.16mm_Horizontal" V 7280 3350 50  0001 C CNN
 F 3 "~" H 7350 3350 50  0001 C CNN
 	1    7350 3350
@@
 $EndComp
 Wire Wire Line
-	6400 4800 7250 4800
-Wire Wire Line
-	7650 4800 7650 4600
-Connection ~ 6400 4800
-Wire Wire Line
-	6400 4800 6400 4700
-Wire Wire Line
-	7250 4600 7250 4800
-Connection ~ 7250 4800
-Wire Wire Line
-	7250 4800 7650 4800
-Wire Wire Line
 	7250 4300 7250 4050
 Wire Wire Line
@@
 F 0 "R17" H 9020 4696 50  0000 L CNN
 F 1 "R" H 9020 4605 50  0000 L CNN
-F 2 "" V 8880 4650 50  0001 C CNN
+F 2 "CmpAmpliAudio:R_Axial_DIN0207_L6.3mm_D2.5mm_P10.16mm_Horizontal" V 8880 4650 50  0001 C CNN
 F 3 "~" H 8950 4650 50  0001 C CNN
 	1    8950 4650
@@
 F 0 "R16" H 9520 3996 50  0000 L CNN
 F 1 "R" H 9520 3905 50  0000 L CNN
-F 2 "" V 9380 3950 50  0001 C CNN
+F 2 "CmpAmpliAudio:R_Axial_DIN0207_L6.3mm_D2.5mm_P10.16mm_Horizontal" V 9380 3950 50  0001 C CNN
 F 3 "~" H 9450 3950 50  0001 C CNN
 	1    9450 3950
@@
 	9450 3300 9450 3450
 Connection ~ 9450 3450
+$Comp
+L be-elec:Relay_1CT U1
+U 1 1 605D271C
+P 8500 3650
+F 0 "U1" H 9050 4517 50  0000 C CNN
+F 1 "Relay_1CT" H 9050 4426 50  0000 C CNN
+F 2 "BE_Elec:Relay_1CT" H 8500 3650 50  0001 C CNN
+F 3 "" H 8500 3650 50  0001 C CNN
+	1    8500 3650
+	1    0    0    -1
+$EndComp
+Wire Wire Line
+	6400 4700 6400 4850
+Wire Wire Line
+	6400 4850 7250 4850
+Wire Wire Line
+	7650 4600 7650 4850
+Connection ~ 6400 4850
+Wire Wire Line
+	7250 4600 7250 4850
+Connection ~ 7250 4850
+Wire Wire Line
+	7250 4850 7650 4850
 $EndSCHEMATC

Commit message: --all
Connections:
- net -12V: now also C3.2
- net GND: no longer C3.2
- net at Q8.2 (C), Q9.3 (B), RV1.1: now also Q6.3 (C); no longer Q6.1 (E)
- net at R7.2: now also Q6.1 (E); no longer Q6.3 (C)
Changed lines of the file:
@@
 	4800 2600 4650 2600
-$Comp
-L Device:Q_PNP_EBC Q6
-U 1 1 605D918E
-P 5000 1950
-F 0 "Q6" H 5190 1996 50  0000 L CNN
-F 1 "2N2907" H 5190 1905 50  0000 L CNN
-F 2 "CmpAmpliAudio:TO-18-3" H 5200 2050 50  0001 C CNN
-F 3 "~" H 5000 1950 50  0001 C CNN
-	1    5000 1950
-	1    0    0    -1
-$EndComp
 $Comp
 L Device:R R7
@@
 	1    0    0    -1
 $EndComp
-$Comp
-L power:GND #PWR0117
-U 1 1 606FD7BB
-P 9450 4950
-F 0 "#PWR0117" H 9450 4700 50  0001 C CNN
-F 1 "GND" H 9455 4777 50  0000 C CNN
-F 2 "" H 9450 4950 50  0001 C CNN
-F 3 "" H 9450 4950 50  0001 C CNN
-	1    9450 4950
-	1    0    0    -1
-$EndComp
 Wire Wire Line
 	9450 3800 9450 3450
@@
 Wire Wire Line
 	8550 3850 8550 3450
-Entry Bus Bus
-	4450 4250 4550 4350
 $Comp
 L power:GND #PWR0119
@@
 Wire Wire Line
 	7250 4850 7650 4850
+$Comp
+L power:-12V #PWR0117
+U 1 1 60728ED9
+P 9450 4950
+F 0 "#PWR0117" H 9450 5050 50  0001 C CNN
+F 1 "-12V" H 9465 5123 50  0000 C CNN
+F 2 "" H 9450 4950 50  0001 C CNN
+F 3 "" H 9450 4950 50  0001 C CNN
+	1    9450 4950
+	-1   0    0    1
+$EndComp
+$Comp
+L Device:Q_PNP_EBC Q6
+U 1 1 6072E0AD
+P 5000 1950
+F 0 "Q6" H 5190 1904 50  0000 L CNN
+F 1 "2N2907" H 5190 1995 50  0000 L CNN
+F 2 "CmpAmpliAudio:TO-18-3" H 5200 2050 50  0001 C CNN
+F 3 "~" H 5000 1950 50  0001 C CNN
+	1    5000 1950
+	1    0    0    1
+$EndComp
 $EndSCHEMATC

Commit message: --all
Parts:
- added D3, D4: 1N4001, Diode_THT:D_DO-41_SOD81_P10.16mm_Horizontal, symbol Diode:1N4001
- C2: value 100n -> C
- R11, R12: footprint CmpAmpliAudio:R_Axial_DIN0207_L6.3mm_D2.5mm_P10.16mm_Horizontal -> CmpAmpliAudio:R_Axial_DIN0516_L15.5mm_D5.0mm_P20.32mm_Horizontal
- RV1, RV2: footprint CmpAmpliAudio:R_Axial_DIN0516_L15.5mm_D5.0mm_P20.32mm_Horizontal -> CmpAmpliAudio:Potentiometer_Bourns_3296W_Vertical
Connections:
- net +12V: now also D3.1 (K)
- net -12V: now also D4.2 (A)
- net GND: now also D3.2 (A), D4.1 (K)
Changed lines of the file:
@@
 encoding utf-8
 Sheet 1 1
-Title ""
+Title "Amplificateur Audio"
 Date ""
 Rev ""
-Comp ""
+Comp "Tom Jullien, Augustin Galloo"
 Comment1 ""
 Comment2 ""
@@
 $EndComp
 $Comp
-L power:GND #PWR0102
-U 1 1 60597BD9
-P 3150 6650
-F 0 "#PWR0102" H 3150 6400 50  0001 C CNN
-F 1 "GND" H 3155 6477 50  0000 C CNN
-F 2 "" H 3150 6650 50  0001 C CNN
-F 3 "" H 3150 6650 50  0001 C CNN
-	1    3150 6650
-	1    0    0    -1
-$EndComp
-$Comp
 L power:+12V #PWR0103
 U 1 1 60598403
@@
 	1150 6350 2250 6350
 Wire Wire Line
-	3150 6350 3150 6650
-Wire Wire Line
 	2250 6550 2250 6350
 Connection ~ 2250 6350
@@
 	2650 6550 2650 6350
 Connection ~ 2650 6350
-Wire Wire Line
-	2650 6350 3150 6350
 Wire Wire Line
 	2650 6350 2650 6200
@@
 P 4400 3250
 F 0 "C2" H 4515 3296 50  0000 L CNN
-F 1 "100n" H 4515 3205 50  0000 L CNN
+F 1 "C" H 4515 3205 50  0000 L CNN
 F 2 "CmpAmpliAudio:C_Rect_L7.2mm_W3.5mm_P5.00mm_FKS2_FKP2_MKS2_MKP2" H 4438 3100 50  0001 C CNN
 F 3 "~" H 4400 3250 50  0001 C CNN
@@
 Wire Wire Line
 	5100 2950 5100 2800
-$Comp
-L Device:R_POT RV1
-U 1 1 605D032E
-P 4500 2600
-F 0 "RV1" H 4431 2646 50  0000 R CNN
-F 1 "R_POT" H 4431 2555 50  0000 R CNN
-F 2 "CmpAmpliAudio:R_Axial_DIN0516_L15.5mm_D5.0mm_P20.32mm_Horizontal" H 4500 2600 50  0001 C CNN
-F 3 "~" H 4500 2600 50  0001 C CNN
-	1    4500 2600
-	1    0    0    -1
-$EndComp
 Wire Wire Line
 	4500 2750 4500 2950
@@
 F 0 "RV2" H 3880 2904 50  0000 R CNN
 F 1 "R_POT" H 3880 2995 50  0000 R CNN
-F 2 "CmpAmpliAudio:R_Axial_DIN0516_L15.5mm_D5.0mm_P20.32mm_Horizontal" H 3950 2950 50  0001 C CNN
+F 2 "CmpAmpliAudio:Potentiometer_Bourns_3296W_Vertical" H 3950 2950 50  0001 C CNN
 F 3 "~" H 3950 2950 50  0001 C CNN
 	1    3950 2950
@@
 	5100 2150 5100 2200
 Wire Wire Line
-	4500 2500 4500 2450
-Wire Wire Line
 	4500 2350 5100 2350
-Connection ~ 4500 2450
-Wire Wire Line
-	4500 2450 4500 2350
 Connection ~ 5100 2350
 Wire Wire Line
@@
 F 0 "R11" H 6470 2846 50  0000 L CNN
 F 1 "R" H 6470 2755 50  0000 L CNN
-F 2 "CmpAmpliAudio:R_Axial_DIN0207_L6.3mm_D2.5mm_P10.16mm_Horizontal" V 6330 2800 50  0001 C CNN
+F 2 "CmpAmpliAudio:R_Axial_DIN0516_L15.5mm_D5.0mm_P20.32mm_Horizontal" V 6330 2800 50  0001 C CNN
 F 3 "~" H 6400 2800 50  0001 C CNN
 	1    6400 2800
@@
 F 0 "R12" H 6470 3346 50  0000 L CNN
 F 1 "R" H 6470 3255 50  0000 L CNN
-F 2 "CmpAmpliAudio:R_Axial_DIN0207_L6.3mm_D2.5mm_P10.16mm_Horizontal" V 6330 3300 50  0001 C CNN
+F 2 "CmpAmpliAudio:R_Axial_DIN0516_L15.5mm_D5.0mm_P20.32mm_Horizontal" V 6330 3300 50  0001 C CNN
 F 3 "~" H 6400 3300 50  0001 C CNN
 	1    6400 3300
@@
 	1    0    0    1
 $EndComp
+$Comp
+L Diode:1N4001 D3
+U 1 1 6073DFD1
+P 3100 6050
+F 0 "D3" V 3054 6130 50  0000 L CNN
+F 1 "1N4001" V 3145 6130 50  0000 L CNN
+F 2 "Diode_THT:D_DO-41_SOD81_P10.16mm_Horizontal" H 3100 5875 50  0001 C CNN
+F 3 "http://www.vishay.com/docs/88503/1n4001.pdf" H 3100 6050 50  0001 C CNN
+	1    3100 6050
+	0    1    1    0
+$EndComp
+$Comp
+L Diode:1N4001 D4
+U 1 1 6073FEE5
+P 3100 6700
+F 0 "D4" V 3054 6780 50  0000 L CNN
+F 1 "1N4001" V 3145 6780 50  0000 L CNN
+F 2 "Diode_THT:D_DO-41_SOD81_P10.16mm_Horizontal" H 3100 6525 50  0001 C CNN
+F 3 "http://www.vishay.com/docs/88503/1n4001.pdf" H 3100 6700 50  0001 C CNN
+	1    3100 6700
+	0    1    1    0
+$EndComp
+Wire Wire Line
+	2650 6350 3100 6350
+Wire Wire Line
+	3100 6350 3100 6200
+Wire Wire Line
+	3100 6550 3100 6350
+Connection ~ 3100 6350
+Wire Wire Line
+	3100 5900 3100 5400
+Wire Wire Line
+	3100 5400 2650 5400
+Connection ~ 2650 5400
+Wire Wire Line
+	3100 6850 3100 7050
+Wire Wire Line
+	3100 7050 2650 7050
+Connection ~ 2650 7050
+$Comp
+L power:GND #PWR0102
+U 1 1 6077786D
+P 3750 6600
+F 0 "#PWR0102" H 3750 6350 50  0001 C CNN
+F 1 "GND" H 3755 6427 50  0000 C CNN
+F 2 "" H 3750 6600 50  0001 C CNN
+F 3 "" H 3750 6600 50  0001 C CNN
+	1    3750 6600
+	1    0    0    -1
+$EndComp
+Wire Wire Line
+	3750 6350 3750 6600
+Wire Wire Line
+	3100 6350 3750 6350
+Wire Wire Line
+	4500 2350 4500 2450
+$Comp
+L Device:R_POT RV1
+U 1 1 607C81F8
+P 4500 2600
+F 0 "RV1" H 4431 2646 50  0000 R CNN
+F 1 "R_POT" H 4431 2555 50  0000 R CNN
+F 2 "CmpAmpliAudio:Potentiometer_Bourns_3296W_Vertical" H 4500 2600 50  0001 C CNN
+F 3 "~" H 4500 2600 50  0001 C CNN
+	1    4500 2600
+	1    0    0    -1
+$EndComp
+Connection ~ 4500 2450
+Wire Wire Line
+	4500 2450 4500 2500
 $EndSCHEMATC

Commit message: Mise à jour netlist et dernières modifications de placement.
Parts:
- Q13: footprint CmpAmpliAudio:TO-92_Inline_Wide -> CmpAmpliAudio:TO-18-3
Changed lines of the file:
@@
 F 0 "Q13" H 8841 4296 50  0000 L CNN
 F 1 "2N222" H 8841 4205 50  0000 L CNN
-F 2 "CmpAmpliAudio:TO-92_Inline_Wide" H 8850 4350 50  0001 C CNN
+F 2 "CmpAmpliAudio:TO-18-3" H 8850 4350 50  0001 C CNN
 F 3 "~" H 8650 4250 50  0001 C CNN
 	1    8650 4250

Commit message: bonne lib, pistes top, texte
Parts:
- C1, C3, C4, C6: footprint CmpAmpliAudio:CP_Radial_D8.0mm_P5.00mm -> TR_MaLib_Ampli_2021:CP_Radial_D8.0mm_P5.00mm
- C10, C8: footprint CmpAmpliAudio:CP_Radial_D12.5mm_P5.00mm -> TR_MaLib_Ampli_2021:CP_Radial_D12.5mm_P5.00mm
- C11, C2, C5, C7, C9: footprint CmpAmpliAudio:C_Rect_L7.2mm_W3.5mm_P5.00mm_FKS2_FKP2_MKS2_MKP2 -> TR_MaLib_Ampli_2021:C_Rect_L7.2mm_W3.5mm_P5.00mm_FKS2_FKP2_MKS2_MKP2
- D1, D2, Dz1: footprint CmpAmpliAudio:D_DO-35_SOD27_P10.16mm_Horizontal -> TR_MaLib_Ampli_2021:D_DO-35_SOD27_P10.16mm_Horizontal
- HS1, HS2: footprint CmpAmpliAudio:Heatsink_Fischer_SK104-STC-STIC_35x13mm_2xDrill2.5mm -> TR_MaLib_Ampli_2021:Heatsink_Fischer_SK104-STC-STIC_35x13mm_2xDrill2.5mm
- J2: footprint CmpAmpliAudio:PhoenixContact_MSTBVA_2,5_2-G-5,08_1x02_P5.08mm_Vertical -> TR_MaLib_Ampli_2021:PhoenixContact_MSTBVA_2,5_2-G-5,08_1x02_P5.08mm_Vertical
- J3: footprint CmpAmpliAudio:PhoenixContact_MSTBVA_2,5_3-G-5,08_1x03_P5.08mm_Vertical -> TR_MaLib_Ampli_2021:PhoenixContact_MSTBVA_2,5_3-G-5,08_1x03_P5.08mm_Vertical
- Q1, Q13, Q2, Q3, Q4, Q5, Q6, Q7: footprint CmpAmpliAudio:TO-18-3 -> TR_MaLib_Ampli_2021:TO-18-3
- Q10, Q12: footprint CmpAmpliAudio:TO-220-3_Vertical -> TR_MaLib_Ampli_2021:TO-220-3_Vertical
- Q11, Q8, Q9: footprint CmpAmpliAudio:TO-126-3_Vertical -> TR_MaLib_Ampli_2021:TO-126-3_Vertical
- R1, R10, R13, R14, R15, R16, R17, R2, R3, R4, R5, R6, R7, R8, R9: footprint CmpAmpliAudio:R_Axial_DIN0207_L6.3mm_D2.5mm_P10.16mm_Horizontal -> TR_MaLib_Ampli_2021:R_Axial_DIN0207_L6.3mm_D2.5mm_P10.16mm_Horizontal
- R11, R12: footprint CmpAmpliAudio:R_Axial_DIN0516_L15.5mm_D5.0mm_P20.32mm_Horizontal -> TR_MaLib_Ampli_2021:R_Axial_DIN0516_L15.5mm_D5.0mm_P20.32mm_Horizontal
- RV1, RV2: footprint CmpAmpliAudio:Potentiometer_Bourns_3296W_Vertical -> TR_MaLib_Ampli_2021:Potentiometer_Bourns_3296W_Vertical
- U2: footprint CmpAmpliAudio:Jack_35RAPC2AV -> TR_MaLib_Ampli_2021:Jack_35RAPC2AV
